File: project/jt.kicad_sch (KiCad schematic)
At the start: 2 parts, among them J2 Raspberry_Pi_2_3

Commit message: Add all the RUNs
Connections:
- net at J2.2 (5V), J2.4 (5V): now also A1.40 (VBUS)
Changed lines of the file:
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@@
+		)
+	)
+	(wire
+		(pts
+			(xy 181.61 24.13) (xy 181.61 33.02)
+		)
+		(stroke
+			(width 0)
+			(type default)
+		)
+	)
+	(wire
+		(pts
+			(xy 85.09 24.13) (xy 181.61 24.13)
+		)
+		(stroke
+			(width 0)
+			(type default)
+		)
+	)
+	(wire
+		(pts
+			(xy 85.09 38.1) (xy 85.09 24.13)
+		)
+		(stroke
+			(width 0)
+			(type default)
 		)
 	)
